File: src/STM32-Pedal/audio_codec.kicad_sch (KiCad schematic)
At the start: 48 parts, among them U501 CS4272, U502 OPA2320, U503 OPA2320, Y501 ASFL1-12.288MHZ-EC-T

Commit message: Schematic - 3.3v, stm32 progress, usb-c
Changed lines of the file:
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@@
 	)
 	(hierarchical_label "ANALOG_OUT"
-		(shape input)
+		(shape output)
 		(at 251.46 143.51 0)
 		(effects
