File: src/STM32-Pedal/power.kicad_sch (KiCad schematic)
At the start: 2 parts, among them U301 TPS7A2450DBVR, U302 AP63203WU

Commit message: Schematic - 3.3v, stm32 progress, usb-c
Parts:
- removed U302: AP63203WU, Package_TO_SOT_SMD:TSOT-23-6, symbol Regulator_Switching:AP63203WU
- added C301: 10uF, Package_TO_SOT_SMD:SOT-23-6, symbol Device:C_Small
- added C302: 100nF, Package_TO_SOT_SMD:SOT-23-6, symbol Device:C_Small
- added C303, C304: 22uF, symbol Device:C
- added L301: 4.7uH, Package_TO_SOT_SMD:TSOT-23-6_HandSoldering, symbol Device:L
- added R301: 93.1k, symbol Device:R_Small_US
- added R302: 30.1k, symbol Device:R_Small_US
- added U302: AP63301WU-7, Package_TO_SOT_SMD:TSOT-23-6_HandSoldering, symbol symlib:AP63301WU-7
Connections:
- net +3.3V: now also C303.1, C304.1, L301.2, R301.1
- net +9V: now also C301.2, U302.2 (EN), U302.3 (VIN)
- net GND: now also C301.1, C303.2, C304.2, R302.2, U302.4 (GND)
- new net: R301.2, R302.1, U302.1 (FB)
- new net: C302.2, L301.1, U302.5 (SW)
- new net: C302.1, U302.6 (BST)
Other:
- note added: "16V ceramic"
- note added: "X7R/X5R, >=10V"
- note added: "shielded power inductor >=4.5A saturation current 4A RMS rating low dc resistance close to BST/SW feedback away from switching"
- moved on the sheet: U301
