File: src/STM32-Pedal/connectors.kicad_sch (KiCad schematic)
At the start: 3 parts, among them J201 AudioJack2, J202 AudioJack2, J203 Barrel_Jack

Commit message: Schematic - 3.3v, stm32 progress, usb-c
Parts:
- added C23: 100nF, Package_TO_SOT_SMD:SOT-23-6, symbol Device:C
- added J204: USB_C_Receptacle_USB2.0_16P, Connector:Tag-Connect_TC2030-IDC-FP_2x03_P1.27mm_Vertical, symbol Connector:USB_C_Receptacle_USB2.0_16P
- added R5, R6: 5.1k, symbol Device:R_US
- added U201: USBLC6-2SC6, Package_TO_SOT_SMD:SOT-23-6, symbol Power_Protection:USBLC6-2SC6
Connections:
- net GND: now also C23.2, J204.A1 (GND), J204.A12 (GND), J204.B1 (GND), J204.B12 (GND), J204.SH (SHIELD), R5.2, R6.2, U201.2 (GND)
- new net: J204.A5 (CC1), R6.1
- new net: J204.B5 (CC2), R5.1
- new net D+: J204.A6 (D+), J204.B6 (D+), U201.1 (I/O1)
- new net D-: J204.A7 (D-), J204.B7 (D-), U201.3 (I/O2)
- new net USB_DM: U201.4 (I/O2)
- new net USB_DP: U201.6 (I/O1)
- new net USB_VBUS: C23.1, J204.A4 (VBUS), J204.A9 (VBUS), J204.B4 (VBUS), J204.B9 (VBUS), U201.5 (VBUS)
- no-connect marks 0 -> 2

Commit message: Schematic: bypass relay, cleaning up input stage
Parts:
- C23: footprint Package_TO_SOT_SMD:SOT-23-6 -> Capacitor_SMD:C_0603_1608Metric_Pad1.08x0.95mm_HandSolder
- J201, J202: footprint Connector_Audio:Jack_6.35mm_Neutrik_NMJ4HFD2_Horizontal -> (none)
- J204: footprint Connector:Tag-Connect_TC2030-IDC-FP_2x03_P1.27mm_Vertical -> (none)
- R5, R6: footprint (none) -> Resistor_SMD:R_0603_1608Metric_Pad0.98x0.95mm_HandSolder
Other:
- note added: "CENTER NEGATIVE"
- note added: "USB-C"
- moved on the sheet: J204, R5, R6, U201
