File: src/STM32-Pedal/input_stage.kicad_sch (KiCad schematic)
At the start: 12 parts, among them U401 OPA2134

Commit message: Schematic - 3.3v, stm32 progress, usb-c
Connections:
- net VCC is gone; now on net +9V: R401.2
Other:
- note added: "SENSITIVE ANALOG"
- note removed: "2ND ORDER SALLEN-KEY LOW PASS"
- note removed: "BIAS"
- note removed: "BUFFER - OPA134"
- note removed: "IN"
- note removed: "VCC BIAS"
Changed lines of the file:
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@@
 	(paper "USLetter")
 	(rectangle
-		(start 25.4 73.66)
+		(start 90.17 73.66)
 		(end 255.27 130.81)
 		(stroke
 			(width 0)
-			(type solid)
+			(type dash)
 			(color 255 0 0 1)
 		)
@@
 		)
 	)
-	(text "BIAS"
+	(text "SENSITIVE ANALOG"
 		(exclude_from_sim no)
-		(at 109.22 90.17 0)
+		(at 108.458 69.088 0)
 		(effects
 			(font
-				(size 1.27 1.27)
+				(size 1.905 1.905)
 				(color 255 0 0 1)
 			)
-		)
-	)
-	(text "IN"
-		(exclude_from_sim no)
-		(at 97.79 98.044 0)
-		(effects
-			(font
-				(size 1.27 1.27)
-				(color 255 0 0 1)
-			)
-		)
-	)
-	(text "BUFFER - OPA134"
-		(exclude_from_sim no)
-		(at 139.446 92.202 0)
-		(effects
-			(font
-				(size 1.27 1.27)
-				(color 255 0 0 1)
-			)
-		)
-	)
-	(text "2ND ORDER SALLEN-KEY LOW PASS"
-		(exclude_from_sim no)
-		(at 212.09 79.756 0)
-		(effects
-			(font
-				(size 1.27 1.27)
-				(color 255 0 0 1)
-			)
-		)
-	)
-	(text "BIAS"
-		(exclude_from_sim no)
-		(at 162.052 93.218 0)
-		(effects
-			(font
-				(size 1.27 1.27)
-				(color 255 0 0 1)
-			)
-		)
-	)
-	(text "VCC BIAS"
-		(exclude_from_sim no)
-		(at 58.928 105.664 0)
-		(effects
-			(font
-				(size 1.27 1.27)
-				(color 255 0 0 1)
-			)
+			(justify left top)
 		)
 	)
@@
 	(symbol
 		(lib_id "power:+9V")
+		(at 44.45 87.63 0)
+		(unit 1)
+		(body_style 1)
+		(exclude_from_sim no)
+		(in_bom yes)
+		(on_board yes)
+		(in_pos_files yes)
+		(dnp no)
+		(fields_autoplaced yes)
+		(property "Reference" "#PWR088"
+			(at 44.45 91.44 0)
+			(hide yes)
+			(show_name no)
+			(do_not_autoplace no)
+			(effects
+				(font
+					(size 1.27 1.27)
+				)
+			)
+		)
+		(property "Value" "+9V"
+			(at 44.45 82.55 0)
+			(show_name no)
+			(do_not_autoplace no)
+			(effects
+				(font
+					(size 1.27 1.27)
+				)
+			)
+		)
+		(property "Footprint" ""
+			(at 44.45 87.63 0)
+			(hide yes)
+			(show_name no)
+			(do_not_autoplace no)
+			(effects
+				(font
+					(size 1.27 1.27)
+				)
+			)
+		)
+		(property "Datasheet" ""
+			(at 44.45 87.63 0)
+			(hide yes)
+			(show_name no)
+			(do_not_autoplace no)
+			(effects
+				(font
+					(size 1.27 1.27)
+				)
+			)
+		)
+		(property "Description" "Power symbol creates a global label with name \"+9V\""
+			(at 44.45 87.63 0)
+			(hide yes)
+			(show_name no)
+			(do_not_autoplace no)
+			(effects
+				(font
+					(size 1.27 1.27)
+				)
+			)
+		)
+		(pin "1"
+		)
+		(instances
+			(project "STM32-Pedal"
+				(path "/a4106809-e56d-4105-b188-893816df5641/20c42f7e-5ce7-467e-a6d2-62bc3fc539c0"
+					(reference "#PWR088")
+					(unit 1)
+				)
+			)
+		)
+	)
+	(symbol
+		(lib_id "power:+9V")
 		(at 73.66 87.63 0)
 		(unit 1)
@@
 					(unit 1)
 				)
-			)
-		)
-	)
-	(symbol
-		(lib_id "power:VCC")
-		(at 44.45 87.63 0)
-		(unit 1)
-		(body_style 1)
-		(exclude_from_sim no)
-		(in_bom yes)
-		(on_board yes)
-		(in_pos_files yes)
-		(dnp no)
-		(fields_autoplaced yes)
-		(property "Reference" "#PWR03"
-			(at 44.45 91.44 0)
-			(hide yes)
-			(show_name no)
-			(do_not_autoplace no)
-			(effects
-				(font
-					(size 1.27 1.27)
-				)
-			)
-		)
-		(property "Value" "VCC"
-			(at 44.45 82.55 0)
-			(show_name no)
-			(do_not_autoplace no)
-			(effects
-				(font
-					(size 1.27 1.27)
-				)
-			)
-		)
-		(property "Footprint" "Package_QFP:TQFP-44_10x10mm_P0.8mm"
-			(at 44.45 87.63 0)
-			(hide yes)
-			(show_name no)
-			(do_not_autoplace no)
-			(effects
-				(font
-					(size 1.27 1.27)
-				)
-			)
-		)
-		(property "Datasheet" ""
-			(at 44.45 87.63 0)
-			(hide yes)
-			(show_name no)
-			(do_not_autoplace no)
-			(effects
-				(font
-					(size 1.27 1.27)
-				)
-			)
-		)
-		(property "Description" "Power symbol creates a global label with name \"VCC\""
-			(at 44.45 87.63 0)
-			(hide yes)
-			(show_name no)
-			(do_not_autoplace no)
-			(effects
-				(font
-					(size 1.27 1.27)
-				)
-			)
-		)
-		(pin "1"
-		)
-		(instances
-			(project "STM32-Pedal"
-				(path "/a4106809-e56d-4105-b188-893816df5641/20c42f7e-5ce7-467e-a6d2-62bc3fc539c0"
-					(reference "#PWR03")
-					(unit 1)
-				)

Commit message: Schematic: bypass relay, cleaning up input stage
Parts:
- added C402: 4.7uF, Capacitor_SMD:C_0805_2012Metric_Pad1.18x1.45mm_HandSolder, symbol Device:C
- added C403: 100nF, Capacitor_SMD:C_0603_1608Metric_Pad1.08x0.95mm_HandSolder, symbol Device:C
- added R403: 2.2M, Resistor_SMD:R_0603_1608Metric_Pad0.98x0.95mm_HandSolder, symbol Device:R_US
- C401: footprint (none) -> Capacitor_SMD:C_0805_2012Metric_Pad1.18x1.45mm_HandSolder
- C404: renamed from C402; footprint (none) -> Capacitor_SMD:C_0603_1608Metric_Pad1.08x0.95mm_HandSolder
- C405: renamed from C403; footprint (none) -> Capacitor_SMD:C_0805_2012Metric_Pad1.18x1.45mm_HandSolder
- C406: renamed from C404; footprint (none) -> Capacitor_SMD:C_0603_1608Metric_Pad1.08x0.95mm_HandSolder
- C407: renamed from C405; footprint (none) -> Capacitor_SMD:C_0603_1608Metric_Pad1.08x0.95mm_HandSolder
- R401, R402: footprint (none) -> Resistor_SMD:R_0603_1608Metric_Pad0.98x0.95mm_HandSolder
- R404: renamed from R403; value 100k -> 2.2M; footprint (none) -> Resistor_SMD:R_0603_1608Metric_Pad0.98x0.95mm_HandSolder
- R405: renamed from R404; footprint (none) -> Resistor_SMD:R_0603_1608Metric_Pad0.98x0.95mm_HandSolder
- R406: renamed from R405; value 2.4k -> 3.06k; footprint (none) -> Resistor_SMD:R_0603_1608Metric_Pad0.98x0.95mm_HandSolder
- R407: renamed from R406; value 2.4k -> 3.06k; footprint (none) -> Resistor_SMD:R_0603_1608Metric_Pad0.98x0.95mm_HandSolder
- U401: footprint (none) -> Package_SO:SOIC-8_3.9x4.9mm_P1.27mm
Connections:
- net +9V: now also C402.2, C403.2
- net GND: now also C402.1, C403.1, R403.1
- net +4.5V renamed VBIAS_4V5
- net AUX_IN renamed EFFECT_IN
- net EFFECT_IN: now also R403.2
Other:
- moved on the sheet: C401, C404, C405, C406, C407, R401, R402, R404, R405, R406, R407, U401A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
