File: src/STM32-Pedal/stm32h743.kicad_sch (KiCad schematic)
At the start: 1 part, among them U1 STM32H743ZITx

Commit message: Schematic - 3.3v, stm32 progress, usb-c
Parts:
- removed U1: STM32H743ZITx, Package_QFP:LQFP-144_20x20mm_P0.5mm, symbol MCU_ST_STM32H7:STM32H743ZITx
- added C1, C10, C11, C13, C15, C17, C2, C20, C22, C3, C4, C5, C6, C7, C8, C9: 100nF, symbol Device:C
- added C12: 4.7uF, symbol Device:C_Polarized_US
- added C14, C16, C21: 1uF, symbol Device:C_Polarized_US
- added C18, C19: 2.2uF, symbol Device:C
- added J1: Conn_01x06_Pin, symbol Connector:Conn_01x06_Pin
- added JP2: Jumper_2_Open, symbol Jumper:Jumper_2_Open
- added R1, R2: R_Photo, Sensor:Avago_APDS-9960, symbol Device:R_Photo
- added R3, R4: 10k, symbol Device:R_US
- added R7: 33k, symbol Device:R_US
- added R8: 82k, symbol Device:R_US
- added RV1, RV2, RV3: R_Potentiometer_US, symbol Device:R_Potentiometer_US
- added SW1, SW2, SW3: SW_SPST, symbol Switch:SW_SPST
- added SW4: SW_Push_Open, Package_DFN_QFN:Nordic_AQFN-94-1EP_7x7mm_P0.4mm, symbol Switch:SW_Push_Open
- added U601: STM32H743ZIT6, Package_QFP:LQFP-144_20x20mm_P0.5mm, symbol MCU_ST_STM32H7:STM32H743ZITx
Connections:
- net CODEC_RST: now also U601.56 (PG0)
- net I2C_SCL: now also U601.139 (PB8)
- net I2C_SDA: now also U601.140 (PB9)
- net SAI_CLK: now also U601.4 (PE5)
- net SAI_FRAME_SYNC: now also U601.3 (PE4)
- net SAI_R: now also U601.2 (PE3)
- net SAI_T: now also U601.5 (PE6)
- new net: R7.2, R8.1, U601.101 (PA9)
- new net +3.3V: C1.1, C10.1, C11.1, C12.1, C13.1, C14.1, C15.1, C16.1, C17.1, C2.1, C20.1, C21.1, C3.1, C4.1, C5.1, C6.1, C7.1, C8.1, C9.1, J1.1 (Pin_1), JP2.2 (B), R3.1, U601.108 (VDD), U601.121 (VDD), U601.131 (VDD), U601.143 (PDR_ON), U601.144 (VDD), U601.17 (VDD), U601.30 (VDD), U601.32 (VREF+), U601.33 (VDDA), U601.39 (VDD), U601.52 (VDD), U601.6 (VBAT), U601.62 (VDD), U601.72 (VDD), U601.84 (VDD), U601.95 (VDD33_USB)
- new net BOOT0: JP2.1 (A), R4.1, U601.138 (BOOT0)
- new net GND: C1.2, C10.2, C11.2, C12.2, C13.2, C14.2, C15.2, C16.2, C17.2, C18.2, C19.2, C2.2, C20.2, C21.2, C22.2, C3.2, C4.2, C5.2, C6.2, C7.2, C8.2, C9.2, J1.6 (Pin_6), R4.2, R8.2, SW4.1 (A), U601.107 (VSS), U601.120 (VSS), U601.130 (VSS), U601.16 (VSS), U601.31 (VSSA), U601.38 (VSS), U601.51 (VSS), U601.61 (VSS), U601.83 (VSS), U601.94 (VSS)
- new net NRST: C22.1, J1.4 (Pin_4), R3.2, SW4.2 (B), U601.25 (NRST)
- new net SWCLK: J1.3 (Pin_3), U601.109 (PA14)
- new net SWDIO: J1.2 (Pin_2), U601.105 (PA13)
- new net SWO: J1.5 (Pin_5), U601.133 (PB3)
- new net USB_DM: U601.103 (PA11)
- new net USB_DP: U601.104 (PA12)
- new net USB_VBUS: R7.1
- new net VCAP: C18.1, C19.1, U601.106 (VCAP), U601.71 (VCAP)
Other:
- note added: "Disable VREFBUF in firmware BOOT_ADD1 = 0x1FF0 <- this may depend on bootloader version (might need external clock) SAI1 block A: slave transmitter, async. Recieve ext clock through PE5/PE4 and transmit through PE6 SAI1 block B: slave reciever, internal sync to block A, recieves through PE3 Shares block A clocks internally Audio format: I2S, stereo, 24-bit samples in two 32-bit slots I2C1: PB8/9,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"
- note added: "HSE CRYSTAL ?"
- note added: "PROGRAMMING: 1. Power board from 9V, connect USB-C 2. Close JP2 to pull BOOT0 high 3. Press and release RESET 4. STM32CubeProgrammer: choose USB, refresh and connect, program 5. Open JP2 and RESET again"
- note added: "Panel Mount Controls"
- note added: "Programming Backup"
- note added: "VBAT"
- note added: "VDD Pins"
- note added: "VDD33_USB"
- note added: "VDDA"
- note added: "VREF+"
- note added: "can also add push button to ground"
- note added: "low-esr ceramic X7R or X5R ESR < 100m"

Commit message: Schematic: bypass relay, cleaning up input stage
Changed lines of the file:
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@@
 		)
 	)
-	(text "Disable VREFBUF in firmware\nBOOT_ADD1 = 0x1FF0 <- this may depend on bootloader version\n(might need external clock)\n\nSAI1 block A: slave transmitter, async. Recieve ext clock through PE5/PE4\nand transmit through PE6\n\nSAI1 block B: slave reciever, internal sync to block A, recieves through PE3\nShares block A clocks internally\n\nAudio format: I2S, stereo, 24-bit samples in two 32-bit slots\n\nI2C1: PB8/9, initially 100kHz\n\nPG0: push-pull output, initially low to hold codec in reset"
+	(text "Disable VREFBUF in firmware\nBOOT_ADD1 = 0x1FF0 <- this may depend on bootloader version\n(might need external clock)\n\nSAI1 block A: slave transmitter, async. Recieve ext clock through PE5/PE4\nand transmit through PE6\n\nSAI1 block B: slave reciever, internal sync to block A, recieves through PE3\nShares block A clocks internally\n\nAudio format: I2S, stereo, 24-bit samples in two 32-bit slots\n\nI2C1: PB8/9, initially 100kHz. codec has addr 0x10\n\nPG0: push-pull output, initially low to hold codec in reset"
 		(exclude_from_sim no)
 		(at 91.44 22.352 0)
@@
 		)
 	)
+	(hierarchical_label "BYPASS_BUTTON"
+		(shape input)
+		(at 304.8 161.29 180)
+		(effects
+			(font
+				(size 1.27 1.27)
+			)
+			(justify right)
+		)
+	)
 	(hierarchical_label "SAI_FRAME_SYNC"
 		(shape input)
@@
 	)
 	(hierarchical_label "USB_DP"
-		(shape input)
+		(shape bidirectional)
 		(at 260.35 97.79 0)
 		(effects
@@
 			)
 			(justify left)
+		)
+	)
+	(hierarchical_label "RELAY_CTRL"
+		(shape output)
+		(at 304.8 163.83 180)
+		(effects
+			(font
+				(size 1.27 1.27)
+			)
+			(justify right)
 		)
 	)
@@
 	)
 	(hierarchical_label "USB_DM"
-		(shape input)
+		(shape bidirectional)
 		(at 260.35 95.25 0)
 		(effects
